File: main.sch (EAGLE design)
At the start: 22 parts, among them Y1 16MHz

Commit message: Move vias
Connections:
- net RX_N renamed TX
- net RX_P renamed RX
Changed lines of the file:
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@@
-</segment>
-</net>
-<net name="RX_P" class="0">
-<segment>
-<label x="124.46" y="121.92" size="1.778" layer="95"/>
-<pinref part="U$1" gate="G$1" pin="PD2(RX)"/>
-<wire x1="124.46" y1="121.92" x2="121.92" y2="121.92" width="0.1524" layer="91"/>
-</segment>
-<segment>
-<pinref part="J4" gate="G$1" pin="3"/>
-<wire x1="167.64" y1="96.52" x2="157.48" y2="96.52" width="0.1524" layer="91"/>
-<label x="157.48" y="96.52" size="1.778" layer="95"/>
-</segment>
-</net>
-<net name="RX_N" class="0">
-<segment>
-<label x="124.46" y="119.38" size="1.778" layer="95"/>
-<label x="124.46" y="119.38" size="1.778" layer="95"/>
-<pinref part="U$1" gate="G$1" pin="PD3(TX)"/>
-<wire x1="124.46" y1="119.38" x2="121.92" y2="119.38" width="0.1524" layer="91"/>
-</segment>
-<segment>
-<wire x1="167.64" y1="93.98" x2="157.48" y2="93.98" width="0.1524" layer="91"/>
-<label x="157.48" y="93.98" size="1.778" layer="95"/>
-<pinref part="J4" gate="G$1" pin="4"/>
 </segment>
 </net>
@@
 </segment>
 </net>
+<net name="RX" class="0">
+<segment>
+<label x="124.46" y="121.92" size="1.778" layer="95"/>
+<pinref part="U$1" gate="G$1" pin="PD2(RX)"/>
+<wire x1="124.46" y1="121.92" x2="121.92" y2="121.92" width="0.1524" layer="91"/>
+</segment>
+<segment>
+<pinref part="J4" gate="G$1" pin="3"/>
+<wire x1="167.64" y1="96.52" x2="157.48" y2="96.52" width="0.1524" layer="91"/>
+<label x="157.48" y="96.52" size="1.778" layer="95"/>
+</segment>
+</net>
+<net name="TX" class="0">
+<segment>
+<label x="124.46" y="119.38" size="1.778" layer="95"/>
+<label x="124.46" y="119.38" size="1.778" layer="95"/>
+<pinref part="U$1" gate="G$1" pin="PD3(TX)"/>
+<wire x1="124.46" y1="119.38" x2="121.92" y2="119.38" width="0.1524" layer="91"/>
+</segment>
+<segment>
+<wire x1="167.64" y1="93.98" x2="157.48" y2="93.98" width="0.1524" layer="91"/>
+<label x="157.48" y="93.98" size="1.778" layer="95"/>
+<pinref part="J4" gate="G$1" pin="4"/>
+</segment>
+</net>
